File: 12_imx1062.kicad_sch (KiCad schematic)
At the start: 115 parts, among them J35 TE_4-1734592-0, J42 Conn_01x02, U15 MIMXRT1062DVL6B, U16 UM803RS, U22 UM1663S, Y3 24MHZ, Y4 32.768KHZ

Commit message: mera
Parts:
- removed C112, C114, C116, C117, C118, C120, C122, C123, C124, C125, C126, C127, C128, C129, C153, C155, C156, C158, C159, C193: 0.22uF, Capacitor_SMD:C_0402_1005Metric, symbol Device:C
- removed C113, C115, C121, C135, C143, C144, C147, C152, C204: 4.7uF, Capacitor_SMD:C_0402_1005Metric, symbol Device:C
- removed C119, C141, C194: 1.0uF, Capacitor_SMD:C_0402_1005Metric, symbol Device:C
- removed C130: 22uF, Capacitor_SMD:C_0603_1608Metric, symbol Device:C
- removed C131, C136, C137, C138, C140, C142, C145, C146, C148, C149, C150, C151, C160, C203: 0.1uF, Capacitor_SMD:C_0402_1005Metric, symbol Device:C
- removed C132, C192: 4.7pF, Capacitor_SMD:C_0402_1005Metric, symbol Device:C
- removed C133, C134: 10pF, Capacitor_SMD:C_0402_1005Metric, symbol Device:C
- removed C139: 10uF, Capacitor_SMD:C_0603_1608Metric, symbol Device:C
- removed C154: 33uF, Capacitor_SMD:C_0603_1608Metric, symbol Device:C
- removed C157: 0.47uF, Capacitor_SMD:C_0402_1005Metric, symbol Device:C
- removed C205: 2.2uF, Capacitor_SMD:C_0402_1005Metric, symbol Device:C
- removed D31: PMEG3020EH, Diode_SMD:D_SOD-123F, symbol Device:D_Schottky
- removed J35: TE_4-1734592-0, footprints:TE_4-1734592-0, symbol Connector_Generic:Conn_01x40
- removed J42: Conn_01x02, Connector_PinHeader_2.54mm:PinHeader_1x02_P2.54mm_Vertical, symbol Connector_Generic:Conn_01x02
- removed L12: 10uH, Inductor_SMD:L_APV_APH0620, symbol Device:L
- removed L9: 4.7uH, Inductor_SMD:L_APV_APH0620, symbol Device:L
- removed R109, R140, R141, R142, R143, R144, R145, R168, R172, R173, R183, R220: 0, Resistor_SMD:R_0402_1005Metric, symbol Device:R_US
- removed R110, R170, R191, R193, R196, R198, R207, R208, R209, R210, R213, R214, R215, R216, R217, R218: 10K, Resistor_SMD:R_0402_1005Metric, symbol Device:R_US
- removed R169: 1.5K, Resistor_SMD:R_0402_1005Metric, symbol Device:R_US
- removed R171: 30K, Resistor_SMD:R_0402_1005Metric, symbol Device:R_US
- removed R182, R222: 10, Resistor_SMD:R_0402_1005Metric, symbol Device:R_US
- removed R192, R194, R195, R197, R199, R200, R201, R202, R203, R204, R205, R206, R211, R212: 1K, Resistor_SMD:R_0402_1005Metric, symbol Device:R_US
- removed R221: 100k, Resistor_SMD:R_0402_1005Metric, symbol Device:R_US
- removed TP28, TP29, TP30: TestPoint, TestPoint:TestPoint_Pad_D2.5mm, symbol Connector:TestPoint
- removed U15: MIMXRT1062DVL6B, footprints:BGA196C65P14X14_1000X1000X152N, symbol imxRT:MIMXRT1062DVL6B
- removed U16: UM803RS, Package_TO_SOT_SMD:SOT-23, symbol Power_Supervisor:LM809
- removed U22: UM1663S, Package_TO_SOT_SMD:SOT-23-6, symbol imxRT:UM1663S
- removed Y3: 24MHZ, footprints:OSC_XRCGB24M000F2P29R0, symbol Device:Crystal_GND24
- removed Y4: 32.768KHZ, footprints:CRYSTAL_FC-135 32.7680KA-AG3_EPS, symbol Device:Crystal
Connections:
- no-connect marks 7 -> 0
