File: 14_RAM.kicad_sch (KiCad schematic)
At the start: 11 parts, among them J18 Conn_01x03, J38 RJHSE5380, J39 Conn_01x03, U19 MAX3232, U20 IS42S16160J-6BLI

Commit message: mera
Parts:
- removed C171, C196, C197, C198: 0.1uF, Capacitor_SMD:C_0402_1005Metric, symbol Device:C
- removed J18, J39: Conn_01x03, Connector_PinHeader_2.54mm:PinHeader_1x03_P2.54mm_Vertical, symbol Connector_Generic:Conn_01x03
- removed J38: RJHSE5380, Connector_RJ:RJ45_Amphenol_RJHSE5380, symbol Connector:8P8C_Shielded
- removed R139, R179: 1K, Resistor_SMD:R_0402_1005Metric, symbol Device:R_US
- removed U19: MAX3232, footprints:PW16_TEX, symbol Interface_UART:MAX3232
- removed U20: IS42S16160J-6BLI, footprints:TFBGA-54_8X8_ISI, symbol imxRT:IS42S16160J-6BLI
Connections:
- no-connect marks 3 -> 0
