File: Ethernet.kicad_sch (KiCad schematic)
At the start: 52 parts, among them J36 Conn_02x10_Odd_Even, J37 RJ45_Hanrun_HR911105A_Horizon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, U17 KSZ8081RNBCA-TR, U18 SRV05-4

Commit message: mera
Parts:
- removed C161: 4.7uF, Capacitor_SMD:C_0402_1005Metric, symbol Device:C
- removed C162, C164, C169, C170, C195: 0.1uF, Capacitor_SMD:C_0402_1005Metric, symbol Device:C
- removed C163: 2.2uF, Capacitor_SMD:C_0402_1005Metric, symbol Device:C
- removed C165, C166, C167, C168: 10pF, Capacitor_SMD:C_0402_1005Metric, symbol Device:C
- removed D22, D30: RB521S30, Diode_SMD:D_SOD-523, symbol Device:D_Schottky
- removed FB1: BLM21PG221SN1D, Inductor_SMD:L_0805_2012Metric, symbol Device:FerriteBead
- removed J36: Conn_02x10_Odd_Even, Connector_PinHeader_2.54mm:PinHeader_2x10_P2.54mm_Vertical, symbol Connector_Generic:Conn_02x10_Odd_Even
- removed J37: RJ45_Hanrun_HR911105A_Horizontal, Connector_RJ:RJ45_Hanrun_HR911105A_Horizontal, symbol Connector:RJ45_Hanrun_HR911105A_Horizontal
- removed L10: L_Iron, Inductor_SMD:L_APV_APH0620, symbol Device:L_Iron
- removed R111, R112, R113, R126, R127, R128, R132, R134, R135, R136, R138, R174, R176, R177: 1K, Resistor_SMD:R_0402_1005Metric, symbol Device:R_US
- removed R114, R115, R116, R117, R118, R119, R120, R121: 10K, Resistor_SMD:R_0402_1005Metric, symbol Device:R_US
- removed R122: 6.49K, Resistor_SMD:R_0402_1005Metric, symbol Device:R_US
- removed R123, R124, R125, R129, R130, R131, R133, R137: 4.7K, Resistor_SMD:R_0402_1005Metric, symbol Device:R_US
- removed R175: 100, Resistor_SMD:R_0402_1005Metric, symbol Device:R_US
- removed R178: 0, Resistor_SMD:R_0402_1005Metric, symbol Device:R_US
- removed U17: KSZ8081RNBCA-TR, footprints:QFN50P500X500X100-33N, symbol KSZ8081RNBCA-TR:KSZ8081RNBCA-TR
- removed U18: SRV05-4, Package_TO_SOT_SMD:SOT-23-6, symbol Power_Protection:SRV05-4
Connections:
- no-connect marks 5 -> 0
