File: MotorVending.kicad_sch (KiCad schematic)
At the start: 76 parts, among them J24 68000-202HLF, Q10 PSMN4R2-30MLD, Q11 PSMN4R2-30MLD, Q12 PSMN4R2-30MLD, Q13 PSMN4R2-30MLD, Q14 PSMN4R2-30MLD, Q22 BC817, Q23 PSMN4R2-30MLD, U10 MC34GD3000EP

Commit message: add revision to motor
Parts:
- removed C175, C95: 1000pF, Capacitor_SMD:C_0402_1005Metric, symbol Device:C
- removed C176: 0.1uF, Capacitor_SMD:C_0402_1005Metric, symbol Device:C_Polarized_US
- removed C177, C182, C86, C89, C92, C94: 0.1uF, Capacitor_SMD:C_0402_1005Metric, symbol Device:C
- removed C178, C79, C80: 1uF, Capacitor_SMD:C_0402_1005Metric, symbol Device:C_Polarized_US
- removed C179, C81: 390pF, Capacitor_SMD:C_0402_1005Metric, symbol Device:C_Polarized_US
- removed C180, C84, C85: 390pF, Capacitor_SMD:C_0402_1005Metric, symbol Device:C
- removed C181: 22uF, Resistor_SMD:R_0603_1608Metric, symbol Device:C
- removed C183: 100uF, Resistor_SMD:R_0603_1608Metric, symbol Device:C_Polarized_US
- removed C87, C88, C90, C91, C93: 2.2uF, Capacitor_SMD:C_0402_1005Metric, symbol Device:C
- removed D11, D26: BAS316, Diode_SMD:D_SOD-323, symbol Diode:BAS316
- removed D12, D13, D25: PMEG3020EH, Diode_SMD:D_SOD-123F, symbol Device:D_Schottky
- removed J24: 68000-202HLF, Connector_PinHeader_2.54mm:PinHeader_1x02_P2.54mm_Vertical, symbol Connector_Generic:Conn_01x02
- removed Q10, Q11, Q12, Q13, Q14, Q23: PSMN4R2-30MLD, Package_TO_SOT_SMD:LFPAK33, symbol PSMN4R2-30MLD:PSMN4R2-30MLD_new
- removed Q22: BC817, Package_TO_SOT_SMD:SOT-23, symbol Transistor_BJT:BC817
- removed R156, R78, R79: 10.0K, Resistor_SMD:R_0402_1005Metric, symbol Device:R_US
- removed R157, R66, R67, R70, R73, R75, R77, R81: 1.0K, Resistor_SMD:R_0402_1005Metric, symbol Device:R_US
- removed R158, R58, R60, R61, R63, R64: 22, Resistor_SMD:R_0402_1005Metric, symbol Device:R_US
- removed R159, R161, R74, R76: 4.70K, Resistor_SMD:R_0402_1005Metric, symbol Device:R_US
- removed R160: 0.006, Resistor_SMD:R_0402_1005Metric, symbol Device:R_US
- removed R59, R62, R65, R68, R69, R82: 18K, Resistor_SMD:R_0402_1005Metric, symbol Device:R_US
- removed R71: 75, Resistor_SMD:R_0402_1005Metric, symbol Device:R_US
- removed R80: 220, Resistor_SMD:R_0402_1005Metric, symbol Device:R_US
- removed R92, R93: 0, Resistor_SMD:R_0402_1005Metric, symbol Device:R
- removed TP18: B, TestPoint:TestPoint_Pad_D2.5mm, symbol Connector:TestPoint
- removed TP19: C, TestPoint:TestPoint_Pad_D2.5mm, symbol Connector:TestPoint
- removed TP20: BEMF_B, TestPoint:TestPoint_Pad_D2.5mm, symbol Connector:TestPoint
- removed TP21: BEMF_A, TestPoint:TestPoint_Pad_D2.5mm, symbol Connector:TestPoint
- removed TP26: A, TestPoint:TestPoint_Pad_D2.5mm, symbol Connector:TestPoint
- removed TP27: BEMF_C, TestPoint:TestPoint_Pad_D2.5mm, symbol Connector:TestPoint
- removed U10: MC34GD3000EP, footprints:QFN50P800X800X100-57N, symbol MC34GD3000EP:MC34GD3000EP
