File: 01_MCU.kicad_sch (KiCad schematic)
At the start: 73 parts, among them J19 Conn_01x03, J2 Conn_01x05, Q1 PMBT2222A, Q15 PMBT2222A, Q16 PMBT2222A, Q17 PMBT2222A, Q18 PMBT2222A, Q19 PMBT2222A, Q5 PMBT2222A, U1 MIMXRT1011DAE5A, U2 UM803RS, Y1 32.768KHz, Y2 24MHz

Commit message: add revision to motor
Parts:
- removed D1, D16, D2, D20, D21, D4: 150040GS73240, LED_SMD:LED_0402_1005Metric, symbol Device:LED
- removed Q1, Q15, Q16, Q17, Q18, Q19: PMBT2222A, Package_TO_SOT_SMD:SOT-23, symbol Transistor_BJT:Q_NPN_BEC
- removed R105, R106, R107, R108, R150, R5: 1K, Resistor_SMD:R_0402_1005Metric, symbol Device:R_US
- added C27: 0.22uF_0402, Capacitor_SMD:C_0402_1005Metric, symbol Device:C
- added R8: 1K, Resistor_SMD:R_0402_1005Metric, symbol Device:R_US
- added SW1: SW_SPDT_312, Button_Switch_THT:SW_XKB_DM1-16UC-1, symbol Switch:SW_SPDT_312
- added TP3: Saklar, TestPoint:TestPoint_Pad_D2.5mm, symbol Connector:TestPoint
- C26: renamed from C15; footprint Capacitor_SMD:C_0402_1005Metric -> Capacitor_SMD:C_0603_1608Metric
- renumbered C4 to C1, C6 to C10, C7 to C11, C11 to C12, C8 to C13, C23 to C14, C19 to C15, C24 to C16, C12 to C17, C9 to C18, C10 to C19, C3 to C2, C25 to C20, C13 to C21, C20 to C22, C14 to C23, C21 to C24, C22 to C25, C16 to C28, C30 to C29, C2 to C3, C31 to C30, C32 to C31, C33 to C32, C34 to C33, C35 to C34, C36 to C35, C17 to C36, C18 to C37, C28 to C4, C1 to C6, C29 to C7, C27 to C8, C26 to C9, D3 to D1, J2 to J1, J19 to J2, Q5 to Q1, R2 to R1, R3 to R2, R148 to R3, R1 to R4, R149 to R5, R95 to R6, R94 to R7, TP6 to TP1, TP1 to TP4, U2 to U1, U1 to U2, Y2 to Y1, Y1 to Y2
Connections:
- net +3V3: now also SW1.2 (C)
- net GND: now also C27.2, R8.2
- net BLDC_CS renamed IOMUXC_GPIO_00_LPSPI2_PCS3
- net BLDC_DRV_EN renamed BMBNG_CONN5
- net IOMUXC_GPIO_05_FLEXPWM1_PWM2_B renamed BMBNG_CONN1
- net IOMUXC_GPIO_06_FLEXPWM1_PWM2_A renamed BMBNG_CONN2
- net IOMUXC_GPIO_07_FLEXPWM1_PWM3_B renamed BMBNG_CONN3
- net IOMUXC_GPIO_08_FLEXPWM1_PWM3_A renamed BMBNG_CONN4
- net IOMUXC_GPIO_SD_01_FLEXPWM1_PWM0_B: no longer names the net of U2.75 (GPIO_SD_01)
- net IOMUXC_GPIO_SD_01_FLEXPWM1_PWM0_B: now also C27.1, R8.1, SW1.1 (B), TP3.1
- net IOMUXC_GPIO_SD_02_FLEXPWM1_PWM0_A: no longer names the net of U2.74 (GPIO_SD_02)
- net MC33926_D1: no longer names the net of U2.70 (GPIO_SD_05)
- net MC33926_EN renamed BMBNG_CONN6
- net MC33926_IN1 renamed BMBNG_CONN0
- net MC33926_IN2 renamed BMBNG_CONN7
- no-connect marks 0 -> 1
Other:
- note removed: "BLDC"

Commit message: dad
da
Parts:
- C1: value 1.0uF -> 1uF; Manufacturer_Part_Number (none) -> CL05A105KO5NNNC
- C10, C11, C12, C15, C17, C19, C21, C3, C5, C6: value 0.22uF -> 220nF; Manufacturer_Part_Number (none) -> CL05B224KO5NNNC
- C13, C18, C2, C23, C33, C34, C35: Manufacturer_Part_Number (none) -> CL05A475MP5NRNC
- C14, C22: value 22uF_0603 -> 22uF; Manufacturer_Part_Number (none) -> CL10A226MQ8NRNC
- C16: value 4.7uF_0402 -> 4.7uF; Manufacturer_Part_Number (none) -> CL05A475MP5NRNC
- C20, C24, C25, C27: value 0.22uF_0402 -> 220nF; Manufacturer_Part_Number (none) -> CL05B224KO5NNNC
- C26: Manufacturer_Part_Number (none) -> CL10A226MQ8NRNC
- C28: value 1.0uF_0402 -> 1uF; Manufacturer_Part_Number (none) -> CL05A105KO5NNNC
- C29, C30, C31, C32: Manufacturer_Part_Number (none) -> CS1005X7R104K500NR
- C36: value 10uF_0603 -> 10uF; Manufacturer_Part_Number (none) -> CS1608X5R106M160NRB
- C37: value 100nF_0402 -> 100nF; Manufacturer_Part_Number (none) -> CS1005X7R104K500NR
- C4, C7, C8, C9: Manufacturer_Part_Number (none) -> GRM1555C1H120JA01D
- D1: Manufacturer_Part_Number (none) -> C6210741
- J1, J2, R2, TP1, TP2, TP3, TP4: now not fitted
- L1: Manufacturer_Part_Number (none) -> MLP2016H4R7MT0S1
- Q1: Manufacturer_Part_Number (none) -> PMBT2222A,215
- R1: Manufacturer_Part_Number (none) -> FRC0402F2204TS
- R3, R5, R6, R7: Manufacturer_Part_Number (none) -> RC0402FR-0710KL
- R4: value 30k -> 30K; Manufacturer_Part_Number (none) -> RC0402FR-0730KL
- R8: Manufacturer_Part_Number (none) -> 0402WGF1001TCE
- SW1: Manufacturer_Part_Number (none) -> DM1-16UC-1
- U1: Manufacturer_Part_Number (none) -> UM803RS
- U2: Manufacturer_Part_Number (none) -> MIMXRT1011DAE5A
- Y1: Manufacturer_Part_Number (none) -> XOS20024000LT00351005
- Y2: Manufacturer_Part_Number (none) -> NX3215SA-32.768kHz-EXS00A-MU00202

Commit message: gema
Parts:
- C1, C28:  LCSC Part # (none) -> C29266
- C10, C11, C12, C15, C17, C19, C20, C21, C24, C25, C27, C3, C5, C6:  LCSC Part # (none) -> C16772
- C13, C16, C18, C2, C23, C33, C34, C35:  LCSC Part # (none) -> C23733
- C14, C22, C26:  LCSC Part # (none) -> C59461
- C29, C30, C31, C32, C37:  LCSC Part # (none) -> C77020; Manufacturer_Part_Number CS1005X7R104K500NR -> GRM155R71H104KE14D
- C36:  LCSC Part # (none) -> C194427; Manufacturer_Part_Number CS1608X5R106M160NRB -> GRM188R6YA106MA73D
- C4, C7, C8, C9:  LCSC Part # (none) -> C76948
- D1:  LCSC Part # (none) -> C6210741
- L1:  LCSC Part # (none) -> C383380
- Q1:  LCSC Part # (none) -> C23869
- R1:  LCSC Part # (none) -> C2998080
- R3, R5, R6, R7:  LCSC Part # (none) -> C60490
- R4:  LCSC Part # (none) -> C138008
- R8:  LCSC Part # (none) -> C11702
- SW1:  LCSC Part # (none) -> C466019
- U1:  LCSC Part # (none) -> C620009
- U2:  LCSC Part # (none) -> C1575810
- Y1:  LCSC Part # (none) -> C2965580; Manufacturer_Part_Number XOS20024000LT00351005 -> XL7EL89CKI-111YLC-24M
- Y2:  LCSC Part # (none) -> C7528807; Manufacturer_Part_Number NX3215SA-32.768kHz-EXS00A-MU00202 -> XKXEL89CJI-SUAYLC-32.768K
