File: 11_GPIO_Expander.kicad_sch (KiCad schematic)
At the start: 12 parts, among them J34 BAMBANG_CONNECTOR, U14 PCA9539PW_118

Commit message: add revision to motor
Parts:
- removed R184, R185, R186, R187, R188, R189, R190, R219: 0, Resistor_SMD:R_0402_1005Metric, symbol Device:R
- renumbered J34 to J29, R96 to R92, R4 to R93
Connections:
- net BMBNG_CONN0: no longer U14.13 (IO1_0)
- net BMBNG_CONN1: no longer U14.14 (IO1_1)
- net BMBNG_CONN2: no longer U14.15 (IO1_2)
- net BMBNG_CONN3: no longer U14.16 (IO1_3)
- net BMBNG_CONN4: no longer U14.17 (IO1_4)
- net BMBNG_CONN5: no longer U14.18 (IO1_5)
- net BMBNG_CONN6: no longer U14.19 (IO1_6)
- net BMBNG_CONN7: no longer U14.20 (IO1_7)
- new net MOTOR_DIR: U14.18 (IO1_5)
- new net MOTOR_EN: U14.13 (IO1_0)
- new net MOTOR_M0: U14.16 (IO1_3)
- new net MOTOR_M1: U14.15 (IO1_2)
- new net MOTOR_M2: U14.14 (IO1_1)
- new net MOTOR_RST: U14.19 (IO1_6)
- new net MOTOR_SLP: U14.20 (IO1_7)
- new net MOTOR_STP: U14.17 (IO1_4)

Commit message: del some
Parts:
- renumbered J29 to J30
Changed lines of the file:
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@@
 		(on_board yes)
 		(dnp no)
-		(property "Reference" "J29"
+		(property "Reference" "J30"
 			(at 73.66 127 0)
 			(effects
@@
 			(project ""
 				(path "/0db193be-516d-4409-bb62-b8733a9e8874/ea7bcb6b-3454-456d-bab5-9b7d764b6981"
-					(reference "J29")
+					(reference "J30")
 					(unit 1)
 				)

Commit message: dad
da
Parts:
- J30: now not fitted
- R92, R93: footprint Capacitor_SMD:C_0402_1005Metric -> Resistor_SMD:R_0402_1005Metric; Manufacturer_Part_Number (none) -> RC0402FR-0710KL
- U14: Manufacturer_Part_Number (none) -> PCA9539PW,118
Changed lines of the file:
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@@
 			)
 		)
-		(property "Footprint" "Capacitor_SMD:C_0402_1005Metric"
+		(property "Footprint" "Resistor_SMD:R_0402_1005Metric"
 			(at 145.161 53.594 90)
 			(effects
@@
 			)
 		)
-		(property "Manufacturer_Part_Number" ""
+		(property "Manufacturer_Part_Number" "RC0402FR-0710KL"
 			(at 144.145 53.34 0)
 			(effects
@@
 		)
 		(property "Value2" ""
+			(at 144.145 53.34 0)
+			(effects
+				(font
+					(size 1.27 1.27)
+				)
+			)
+		)
+		(property "partNum" ""
 			(at 144.145 53.34 0)
 			(effects
@@
 		(in_bom yes)
 		(on_board yes)
-		(dnp no)
+		(dnp yes)
 		(property "Reference" "J30"
 			(at 73.66 127 0)
@@
 		)
 		(property "Value2" ""
+			(at 73.66 100.33 0)
+			(effects
+				(font
+					(size 1.27 1.27)
+				)
+			)
+		)
+		(property "partNum" ""
 			(at 73.66 100.33 0)
 			(effects
@@
 			)
 		)
-		(property "Manufacturer_Part_Number" ""
+		(property "Manufacturer_Part_Number" "PCA9539PW,118"
 			(at 123.19 80.01 0)
 			(effects
@@
 		)
 		(property "Value2" ""
+			(at 123.19 80.01 0)
+			(effects
+				(font
+					(size 1.27 1.27)
+				)
+			)
+		)
+		(property "partNum" ""
 			(at 123.19 80.01 0)
 			(effects
@@
 			)
 		)
-		(property "Footprint" "Capacitor_SMD:C_0402_1005Metric"
+		(property "Footprint" "Resistor_SMD:R_0402_1005Metric"
 			(at 72.771 56.769 90)
 			(effects
@@
 			)
 		)
-		(property "Manufacturer_Part_Number" ""
+		(property "Manufacturer_Part_Number" "RC0402FR-0710KL"
 			(at 71.755 56.515 0)
 			(effects
@@
 			(at 71.755 56.515 0)
 			(effects
+				(font
+					(size 1.27 1.27)
+				)
+			)
+		)
+		(property "partNum" ""
+			(at 71.755 56.515 0)
+			(effects

Commit message: gema
Parts:
- R92, R93:  LCSC Part # (none) -> C60490
- U14:  LCSC Part # (none) -> C2687996
Changed lines of the file:
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@@
+			)
+		)
+		(property " LCSC Part #" "C60490"
+			(at 144.145 53.34 0)
+			(effects
+				(font
+					(size 1.27 1.27)
+				)
+				(hide yes)
 			)
 		)
@@
 			)
 		)
+		(property " LCSC Part #" ""
+			(at 73.66 100.33 0)
+			(effects
+				(font
+					(size 1.27 1.27)
+				)
+				(hide yes)
+			)
+		)
 		(pin "11"
 		)
@@
 			)
 		)
+		(property " LCSC Part #" "C2687996"
+			(at 123.19 80.01 0)
+			(effects
+				(font
+					(size 1.27 1.27)
+				)
+				(hide yes)
+			)
+		)
 		(pin "17"
 		)
@@
 			)
 		)
+		(property " LCSC Part #" "C60490"
+			(at 71.755 56.515 0)
+			(effects
+				(font
+					(size 1.27 1.27)
+				)
+				(hide yes)
+			)
+		)
