File: USB.kicad_sch (KiCad schematic)
At the start: 10 parts, among them J15 TYPE-C-31-M-12, Q20 PMBT2222A

Commit message: add revision to motor
Parts:
- renumbered C110 to C38, D18 to D2, D19 to D3, D23 to D4, J15 to J3, Q20 to Q2, R104 to R10, R146 to R12, R103 to R9
Other:
- moved on the sheet: R10

Commit message: dad
da
Parts:
- C38: Manufacturer_Part_Number (none) -> CL10A226MQ8NRNC
- D2, D3: Manufacturer_Part_Number (none) -> PMEG3020EH
- D4: Manufacturer_Part_Number (none) -> C6210741
- J3: Manufacturer_Part_Number (none) -> TYPE-C-31-M-12
- Q2: Manufacturer_Part_Number (none) -> PMBT2222A,215
- R10, R9: Manufacturer_Part_Number (none) -> RC0402FR-075K1L
- R11: Manufacturer_Part_Number (none) -> RC0402FR-072K7L
- R12: Manufacturer_Part_Number (none) -> 0402WGF1001TCE
Changed lines of the file:
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@@
 			)
 		)
-		(property "Manufacturer_Part_Number" ""
+		(property "Manufacturer_Part_Number" "PMBT2222A,215"
 			(at 136.525 69.85 0)
 			(effects
@@
 		)
 		(property "Value2" ""
+			(at 136.525 69.85 0)
+			(effects
+				(font
+					(size 1.27 1.27)
+				)
+			)
+		)
+		(property "partNum" ""
 			(at 136.525 69.85 0)
 			(effects
@@
 			)
 		)
-		(property "Manufacturer_Part_Number" ""
+		(property "Manufacturer_Part_Number" "PMEG3020EH"
 			(at 133.35 43.18 0)
 			(effects
@@
 		)
 		(property "Value2" ""
+			(at 133.35 43.18 0)
+			(effects
+				(font
+					(size 1.27 1.27)
+				)
+			)
+		)
+		(property "partNum" ""
 			(at 133.35 43.18 0)
 			(effects
@@
 			)
 		)
-		(property "Manufacturer_Part_Number" ""
+		(property "Manufacturer_Part_Number" "TYPE-C-31-M-12"
 			(at 64.135 50.165 0)
 			(effects
@@
 		)
 		(property "Value2" ""
+			(at 64.135 50.165 0)
+			(effects
+				(font
+					(size 1.27 1.27)
+				)
+			)
+		)
+		(property "partNum" ""
 			(at 64.135 50.165 0)
 			(effects
@@
 			)
 		)
-		(property "Manufacturer_Part_Number" ""
+		(property "Manufacturer_Part_Number" "CL10A226MQ8NRNC"
 			(at 164.465 40.005 0)
 			(effects
@@
 		)
 		(property "Value2" ""
+			(at 164.465 40.005 0)
+			(effects
+				(font
+					(size 1.27 1.27)
+				)
+			)
+		)
+		(property "partNum" ""
 			(at 164.465 40.005 0)
 			(effects
@@
 			)
 		)
-		(property "Manufacturer_Part_Number" ""
+		(property "Manufacturer_Part_Number" "PMEG3020EH"
 			(at 132.08 32.385 0)
 			(effects
@@
 		)
 		(property "Value2" ""
+			(at 132.08 32.385 0)
+			(effects
+				(font
+					(size 1.27 1.27)
+				)
+			)
+		)
+		(property "partNum" ""
 			(at 132.08 32.385 0)
 			(effects
@@
 			)
 		)
-		(property "Manufacturer_Part_Number" ""
+		(property "Manufacturer_Part_Number" "RC0402FR-075K1L"
 			(at 31.75 67.31 0)
 			(effects
@@
 		)
 		(property "Value2" ""
+			(at 31.75 67.31 0)
+			(effects
+				(font
+					(size 1.27 1.27)
+				)
+			)
+		)
+		(property "partNum" ""
 			(at 31.75 67.31 0)
 			(effects
@@
 			)
 		)
-		(property "Manufacturer_Part_Number" ""
+		(property "Manufacturer_Part_Number" "RC0402FR-072K7L"
 			(at 119.38 48.895 0)
 			(effects
@@
 		)
 		(property "Value2" ""
+			(at 119.38 48.895 0)
+			(effects
+				(font
+					(size 1.27 1.27)
+				)
+			)
+		)
+		(property "partNum" ""
 			(at 119.38 48.895 0)
 			(effects
@@
 			)
 		)
-		(property "Manufacturer_Part_Number" ""
+		(property "Manufacturer_Part_Number" "C6210741"
 			(at 156.21 64.135 0)
 			(effects
@@
 		)
 		(property "Value2" ""
+			(at 156.21 64.135 0)
+			(effects
+				(font
+					(size 1.27 1.27)
+				)
+			)
+		)
+		(property "partNum" ""
 			(at 156.21 64.135 0)
 			(effects
@@
 			)
 		)
-		(property "Manufacturer_Part_Number" ""
+		(property "Manufacturer_Part_Number" "0402WGF1001TCE"
 			(at 146.05 64.135 0)
 			(effects
@@
 		)
 		(property "Value2" ""
+			(at 146.05 64.135 0)
+			(effects
+				(font
+					(size 1.27 1.27)
+				)
+			)
+		)
+		(property "partNum" ""
 			(at 146.05 64.135 0)
 			(effects
@@
 			)
 		)
-		(property "Manufacturer_Part_Number" ""
+		(property "Manufacturer_Part_Number" "RC0402FR-075K1L"
 			(at 96.012 59.182 0)
 			(effects
@@
 			(at 96.012 59.182 0)
 			(effects
+				(font
+					(size 1.27 1.27)
+				)
+			)
+		)
+		(property "partNum" ""
+			(at 96.012 59.182 0)
+			(effects

Commit message: gema
Parts:
- C38:  LCSC Part # (none) -> C59461
- D2, D3:  LCSC Part # (none) -> C167645
- D4:  LCSC Part # (none) -> C6210741
- J3:  LCSC Part # (none) -> C165948
- Q2:  LCSC Part # (none) -> C23869
- R10, R9:  LCSC Part # (none) -> C105872
- R11:  LCSC Part # (none) -> C138017
- R12:  LCSC Part # (none) -> C11702
Changed lines of the file:
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@@
+			)
+		)
+		(property " LCSC Part #" "C23869"
+			(at 136.525 69.85 0)
+			(effects
+				(font
+					(size 1.27 1.27)
+				)
+				(hide yes)
 			)
 		)
@@
 			)
 		)
+		(property " LCSC Part #" "C167645"
+			(at 133.35 43.18 90)
+			(effects
+				(font
+					(size 1.27 1.27)
+				)
+				(hide yes)
+			)
+		)
 		(pin "2"
 		)
@@
 		(on_board yes)
 		(dnp no)
-		(fields_autoplaced yes)
 		(property "Reference" "J3"
 			(at 64.135 32.385 0)
@@
 		)
 		(property "Manufacturer_Part_Number" "TYPE-C-31-M-12"
-			(at 64.135 50.165 0)
+			(at 63.754 28.448 0)
 			(effects
 				(font
@@
 					(size 1.27 1.27)
 				)
+			)
+		)
+		(property " LCSC Part #" "C165948"
+			(at 64.135 50.165 0)
+			(effects
+				(font
+					(size 1.27 1.27)
+				)
+				(hide yes)
 			)
 		)
@@
 			)
 		)
+		(property " LCSC Part #" "C59461"
+			(at 164.465 40.005 0)
+			(effects
+				(font
+					(size 1.27 1.27)
+				)
+				(hide yes)
+			)
+		)
 		(pin "1"
 		)
@@
 			)
 		)
+		(property " LCSC Part #" "C167645"
+			(at 132.08 32.385 90)
+			(effects
+				(font
+					(size 1.27 1.27)
+				)
+				(hide yes)
+			)
+		)
 		(pin "2"
 		)
@@
 			)
 		)
+		(property " LCSC Part #" "C105872"
+			(at 31.75 67.31 90)
+			(effects
+				(font
+					(size 1.27 1.27)
+				)
+				(hide yes)
+			)
+		)
 		(pin "2"
 		)
@@
 					(size 1.27 1.27)
 				)
+			)
+		)
+		(property " LCSC Part #" "C138017"
+			(at 119.38 48.895 90)
+			(effects
+				(font
+					(size 1.27 1.27)
+				)
+				(hide yes)
 			)
 		)
@@
 			)
 		)
+		(property " LCSC Part #" "C6210741"
+			(at 156.21 64.135 0)
+			(effects
+				(font
+					(size 1.27 1.27)
+				)
+				(hide yes)
+			)
+		)
 		(pin "1"
 		)
@@
 			)
 		)
+		(property " LCSC Part #" "C11702"
+			(at 146.05 64.135 90)
+			(effects
+				(font
+					(size 1.27 1.27)
+				)
+				(hide yes)
+			)
+		)
 		(pin "1"
 		)
@@
 			)
 		)
+		(property " LCSC Part #" "C105872"
+			(at 96.012 59.182 90)
+			(effects
+				(font
+					(size 1.27 1.27)
+				)
+				(hide yes)
+			)
+		)
